Commit message: Updating the urdf

File: gavlab_atrv_description/urdf/atrv.urdf.xacro (robot description, xacro)
@@ -24,4 +24,5 @@
   <xacro:property name="chassis_height" value="0.50" />
   <xacro:property name="wheel_radius" value="0.20"/>
+  <xacro:property name="wheel_width" value="0.15"/>
 <!-- xacro macros -->
   <xacro:macro name="default_inertial" params="mass">
@@ -69,14 +70,14 @@
       <xacro:default_inertial mass="1"/>
       <visual>
-        <origin xyz="0 0 ${0.25/2}" rpy="0 0 0" />
+        <origin xyz="0 0 ${wheel_width/2}" rpy="0 0 0" />
         <geometry>
-          <cylinder radius="${wheel_radius}" length="0.25"/>
+          <cylinder radius="${wheel_radius}" length="${wheel_width}"/>
         </geometry>
         <material name="Black"/>
       </visual>
       <collision>
-        <origin xyz="0 0 ${0.25/2}" rpy="0 0 0" />
+        <origin xyz="0 0 ${wheel_width/2}" rpy="0 0 0" />
         <geometry>
-          <cylinder radius="${wheel_radius}" length="0.25"/>
+          <cylinder radius="${wheel_radius}" length="${wheel_width}"/>
         </geometry>
       </collision>
@@ -98,4 +99,29 @@
   <!-- right_rear_wheel_link -->
   <xacro:wheel prefix="right_rear" reflect_x="-1" reflect_y="-1" />
+  <!-- laser_link -->
+  <xacro:property name="laser_radius" value="0.045"/>
+  <xacro:property name="laser_height" value="0.16"/>
+  <link name="laser_link">
+    <xacro:default_inertial mass="3"/>
+    <visual>
+      <origin xyz="0 0 ${0.04-laser_height/2.0}" rpy="0 0 0"/>
+      <geometry>
+        <cylinder radius="${laser_radius}" length="${laser_height}"/>
+      </geometry>
+      <material name="Grey"/>
+    </visual>
+    <collision>
+      <origin xyz="0 0 ${0.04-laser_height/2.0}" rpy="0 0 0"/>
+      <geometry>
+        <cylinder radius="${laser_radius}" length="${laser_height}"/>
+      </geometry>
+    </collision>
+  </link>
+  <!-- base_link -> laser_link -->
+  <joint name="base_laser_joint" type="fixed">
+    <origin xyz="${0.015+laser_radius+chassis_length/2.0} 0 ${0.28-ground_clearance}" rpy="0 0 0"/>
+    <parent link="base_link"/>
+    <child link="laser_link"/>
+  </joint>
   <!-- kinect_link -->
   <link name="kinect_link">

Commit message: ATRV ready for first data collection run

File: gavlab_atrv_description/urdf/atrv.urdf.xacro (robot description, xacro)
@@ -140,8 +140,4 @@
     </collision>
   </link>
-  <link name="kinect_depth_frame"></link>
-  <link name="kinect_depth_optical_frame"></link>
-  <link name="kinect_rgb_frame"></link>
-  <link name="kinect_rgb_optical_frame"></link>
   <!-- base_link -> base_kinect_join -->
   <joint name="base_kinect_joint" type="fixed">
@@ -150,23 +146,10 @@
     <child link="kinect_link"/>
   </joint>
-  <joint name="kinect_depth_joint" type="fixed">
-    <origin xyz="0 0.018 0" rpy="0 0 0" />
-    <parent link="kinect_link" />
-    <child link="kinect_depth_frame" />
-  </joint>
-  <joint name="kinect_depth_optical_joint" type="fixed">
-    <origin xyz="0 0 0" rpy="${-M_PI/2} 0 ${-M_PI/2}"/>
-    <parent link="kinect_depth_frame" />
-    <child link="kinect_depth_optical_frame" />
-  </joint>
-  <joint name="kinect_rgb_joint" type="fixed">
-    <origin xyz="0 -0.005 0" rpy="0 0 0" />
-    <parent link="kinect_link" />
-    <child link="kinect_rgb_frame" />
-  </joint>
-  <joint name="kinect_rgb_optical_joint" type="fixed">
-    <origin xyz="0 0 0" rpy="${-M_PI/2} 0 ${-M_PI/2}"/>
-    <parent link="kinect_rgb_frame" />
-    <child link="kinect_rgb_optical_frame" />
+  <link name="openni_camera"/>
+  <!-- kinect_link -> openni_camera (This is the openni_camera pkg's tf's) -->
+  <joint name="kinect_openni_camera_joint" type="fixed">
+    <origin xyz="0 0 0" rpy="0 0 0"/>
+    <parent link="kinect_link"/>
+    <child link="openni_camera"/>
   </joint>
 </robot>

Commit message: Adding new chassis model for the atrv

File: gavlab_atrv_description/urdf/atrv.urdf.xacro (robot description, xacro)
@@ -8,7 +8,6 @@
   <material name="Black"><color rgba="0.0 0.0 0.0 1.0"/></material>
   <material name="Grey"><color rgba="0.7 0.7 0.7 0.7"/></material>
-  <material name="atrv_orange">
-    <color rgba="0.8 0.16 0.0 1" />
-  </material>
+  <material name="atrv_orange"><color rgba="0.8 0.16 0.0 1" /></material>
+  <material name="clear"><color rgba="0 0 0 0"/></material>
 <!-- xacro parameters -->
   <xacro:property name="M_PI" value="3.14159"/>
@@ -46,14 +45,13 @@
     <xacro:default_inertial mass="80"/>
     <visual>
-      <origin xyz="0 0 ${chassis_height/2.0}" rpy="0 0 0" />
       <geometry>
-        <box size="${chassis_length} ${chassis_width} ${chassis_height}" />
+        <mesh filename="package://gavlab_atrv_description/meshes/atrv_chassis.dae"/>
       </geometry>
-      <material name="atrv_orange" />
+      <!-- <material name="clear"/> -->
     </visual>
     <collision>
       <origin xyz="0 0 ${chassis_height/2.0}" rpy="0 0 0" />
       <geometry>
-        <box size="${chassis_length_bumpers} ${chassis_width} ${chassis_height}" />
+        <box size="${chassis_length} ${chassis_width} ${chassis_height}" />
       </geometry>
     </collision>

Commit message: Updating for fuerte

File: gavlab_atrv_description/urdf/atrv.urdf.xacro (robot description, xacro)
@@ -97,4 +97,11 @@
   <!-- right_rear_wheel_link -->
   <xacro:wheel prefix="right_rear" reflect_x="-1" reflect_y="-1" />
+  <!-- Imu Link -->
+  <link name="imu_frame"/>
+  <joint name="base_imu_joint" type="fixed">
+    <origin xyz="-0.11 0 0.27" rpy="0 0 0"/>
+    <parent link="base_link"/>
+    <child link="imu_frame"/>
+  </joint>
   <!-- laser_link -->
   <xacro:property name="laser_radius" value="0.045"/>
@@ -123,5 +130,5 @@
   </joint>
   <!-- kinect_link -->
-  <link name="kinect_link">
+  <link name="asus_link">
     <xacro:default_inertial mass="0.0001"/>
     <visual>
@@ -142,12 +149,5 @@
     <origin xyz="${(chassis_length/2)-0.19} 0 ${chassis_height+0.13-0.06}" rpy="0 0 0"/>
     <parent link="base_link"/>
-    <child link="kinect_link"/>
-  </joint>
-  <link name="openni_camera"/>
-  <!-- kinect_link -> openni_camera (This is the openni_camera pkg's tf's) -->
-  <joint name="kinect_openni_camera_joint" type="fixed">
-    <origin xyz="0 0 0" rpy="0 0 0"/>
-    <parent link="kinect_link"/>
-    <child link="openni_camera"/>
+    <child link="asus_link"/>
   </joint>
 </robot>

Commit message: Updating launch files and helper scripts

File: gavlab_atrv_description/urdf/atrv.urdf.xacro (robot description, xacro)
@@ -147,5 +147,8 @@
   <!-- base_link -> base_kinect_join -->
   <joint name="base_kinect_joint" type="fixed">
-    <origin xyz="${(chassis_length/2)-0.19} 0 ${chassis_height+0.13-0.06}" rpy="0 0 0"/>
+  <!-- <joint name="base_kinect_joint" type="planar"> -->
+    <origin xyz="${(chassis_length/2)-0.19} 0 ${chassis_height+0.13-0.06}" rpy="0 -0.025 0.04"/>
+    <!-- <axis xyz="0 0 1"/> -->
+    <!-- <limit effort="1" velocity="1" lower="-1" upper="1" /> -->
     <parent link="base_link"/>
     <child link="asus_link"/>

Commit message: updated asus transform to new mount location

File: gavlab_atrv_description/urdf/atrv.urdf.xacro (robot description, xacro)
@@ -148,5 +148,5 @@
   <joint name="base_kinect_joint" type="fixed">
   <!-- <joint name="base_kinect_joint" type="planar"> -->
-    <origin xyz="${(chassis_length/2)-0.19} 0 ${chassis_height+0.13-0.06}" rpy="0 -0.025 0.04"/>
+    <origin xyz="${(chassis_length/2)-0.229} 0 ${chassis_height+0.092}" rpy="0 0 0"/>
     <!-- <axis xyz="0 0 1"/> -->
     <!-- <limit effort="1" velocity="1" lower="-1" upper="1" /> -->

Commit message: changed cmd velocity to ENU convention

File: gavlab_atrv_description/urdf/atrv.urdf.xacro (robot description, xacro)
@@ -148,5 +148,5 @@
   <joint name="base_kinect_joint" type="fixed">
   <!-- <joint name="base_kinect_joint" type="planar"> -->
-    <origin xyz="${(chassis_length/2)-0.229} 0 ${chassis_height+0.092}" rpy="0 0 0"/>
+    <origin xyz="${(chassis_length/2)-0.229} 0 ${chassis_height+0.092}" rpy="0 0 0.04"/>
     <!-- <axis xyz="0 0 1"/> -->
     <!-- <limit effort="1" velocity="1" lower="-1" upper="1" /> -->

Commit message: changes from atrv

File: gavlab_atrv_description/urdf/atrv.urdf.xacro (robot description, xacro)
@@ -37,5 +37,5 @@
   <!-- The frame of the floor directly below the base_link and -->
   <!-- is needed for the navigation stack to work properly -->
-  <link name="base_footprint"></link>
+  <link name="base_footprint"/>  <!-- </link> -->
   <!-- base_link -->
   <!-- The link that is the origin of all of the components of the -->
@@ -59,5 +59,6 @@
   <!-- base_footprint -> base_link -->
   <joint name="base_footprint_joint" type="fixed">
-      <origin xyz="0 0 ${ground_clearance}" rpy="0 0 0"/>
+      <!-- <origin xyz="0 0 ${ground_clearance}" rpy="0 0 0"/> -->
+      <origin xyz="-0.23495 0 ${ground_clearance}" rpy="0 0 0"/>
       <parent link="base_footprint"/>
       <child link="base_link"/>
